Commit message: Geometry completed

File: catkin_ws/src/my_robot/urdf/my_robot.xacro (robot description, xacro)
@@ -31,13 +31,9 @@
     <inertial>
       <mass value="1.0"/>
-      <origin xyz="0.15 0.2 .0125" rpy=" 0 1.5705 1.5705"/>
-      <inertia
-          ixx="0.1" ixy="0" ixz="0"
-          iyy="0.1" iyz="0"
-          izz="0.1"
-      />
+      <origin xyz="0 0 0" rpy=" 0 1.5705 1.5705"/>
+      <inertia ixx="0.1" ixy="0" ixz="0" iyy="0.1" iyz="0" izz="0.1"/>
     </inertial>
     <visual name='front_left_visual'>
-      <origin xyz="0.15 0.2 .0125" rpy=" 0 1.5705 1.5705"/>
+      <origin xyz="0 0 0" rpy=" 0 1.5705 1.5705"/>
       <geometry>
         <cylinder radius="0.1" length="0.1"/>
@@ -45,7 +41,7 @@
     </visual>
     <collision name='front_left_collision'>
-      <origin xyz="0.15 0.2 .0125" rpy=" 0 1.57050 1.5705"/>
+      <origin xyz="0 0 0" rpy=" 0 1.57050 1.5705"/>
       <geometry>
-        cylinder radius="0.1" length="0.1"/>
+        <cylinder radius="0.1" length="0.1"/>
       </geometry>
     </collision>
@@ -55,5 +51,5 @@
     <inertial>
       <mass value="1.0"/>
-      <origin xyz="0.15 -0.2 .0125" rpy=" 0 1.5705 1.5705"/>
+      <origin xyz="0 0 0" rpy=" 0 1.5705 1.5705"/>
       <inertia
           ixx="0.1" ixy="0" ixz="0"
@@ -63,5 +59,5 @@
     </inertial>
     <visual name='front_right_visual'>
-      <origin xyz="0.15 -0.2 .0125" rpy=" 0 1.5705 1.5705 "/>
+      <origin xyz="0 0 0" rpy=" 0 1.5705 1.5705 "/>
       <geometry>
         <cylinder radius="0.1" length="0.1"/>
@@ -69,7 +65,7 @@
     </visual>
     <collision name='front_right_collision'>
-      <origin xyz="0.15 -0.2 .0125" rpy=" 0 1.5705 1.5705"/>
+      <origin xyz="0 0 0" rpy=" 0 1.5705 1.5705"/>
       <geometry>
-        cylinder radius="0.1" length="0.1"/>
+        <cylinder radius="0.1" length="0.1"/>
       </geometry>
     </collision>
@@ -79,13 +75,9 @@
     <inertial>
       <mass value="1.0"/>
-      <origin xyz="-0.15 0.2 .0125" rpy=" 0 1.5705 1.5705"/>
-      <inertia
-          ixx="0.1" ixy="0" ixz="0"
-          iyy="0.1" iyz="0"
-          izz="0.1"
-      />
+      <origin xyz="0 0 0" rpy=" 0 1.5705 1.5705"/>
+      <inertia ixx="0.1" ixy="0" ixz="0" iyy="0.1" iyz="0" izz="0.1"/>
     </inertial>
     <visual name='back_left_visual'>
-      <origin xyz="-0.15 0.2 .0125" rpy=" 0 1.5705 1.5705"/>
+      <origin xyz="0 0 0" rpy=" 0 1.5705 1.5705"/>
       <geometry>
         <cylinder radius="0.1" length="0.1"/>
@@ -93,7 +85,7 @@
     </visual>
     <collision name='back_left_collision'>
-      <origin xyz="-0.15 0.2 .0125" rpy=" 0 1.5705 1.5705"/>
+      <origin xyz="0 0 0 " rpy=" 0 1.5705 1.5705"/>
       <geometry>
-        cylinder radius="0.1" length="0.1"/>
+        <cylinder radius="0.1" length="0.1"/>
       </geometry>
     </collision>
@@ -103,5 +95,5 @@
     <inertial>
       <mass value="1.0"/>
-      <origin xyz="-0.15 -0.2 .0125" rpy=" 1.5705 0 0"/>
+      <origin xyz="0 0 0" rpy=" 1.5705 0 0"/>
       <inertia
           ixx="0.1" ixy="0" ixz="0"
@@ -111,5 +103,5 @@
     </inertial>
     <visual name='back_right_visual'>
-      <origin xyz="-0.15 -0.2 .0125" rpy=" 0 1.5705 1.5705"/>
+      <origin xyz="0 0 0" rpy=" 0 1.5705 1.5705"/>
       <geometry>
         <cylinder radius="0.1" length="0.1"/>
@@ -117,7 +109,27 @@
     </visual>
     <collision name='back_right_collision'>
-      <origin xyz="-0.15 -0.2 .0125" rpy=" 0 1.5705 1.5705"/>
+      <origin xyz="0 0 0" rpy=" 0 1.5705 1.5705"/>
       <geometry>
-        cylinder radius="0.1" length="0.1"/>
+        <cylinder radius="0.1" length="0.1"/>
+      </geometry>
+    </collision>
+   </link>
+   <link name='lidar_base'>
+    <pose>0 0 0.1 0 0 0</pose>
+    <inertial>
+      <mass value="1.0"/>
+      <origin xyz="0 0 0" rpy=" 0 0 0"/>
+      <inertia ixx="0.1" ixy="0" ixz="0" iyy="0.1" iyz="0" izz="0.1"/>
+    </inertial>
+    <visual name='lidar_base_visual'>
+      <origin xyz="0 0 0" rpy=" 0 0 0"/>
+      <geometry>
+        <cylinder radius="0.1" length="0.1"/>
+      </geometry>
+    </visual>
+    <collision name='lidar_base_collision'>
+      <origin xyz="0 0 0" rpy=" 0 0 0"/>
+      <geometry>
+        <cylinder radius="0.1" length="0.1"/>
       </geometry>
     </collision>
@@ -128,4 +140,6 @@
     <child link="front_left_wheel"/>
     <axis xyz="0 1 0"/>
+    <limit effort="10000" velocity="1000"/>
+    <dynamics damping="1.0" friction="1.0"/>
   </joint>
   <joint name="joint_1" type="revolute">
@@ -134,16 +148,28 @@
     <child link="front_right_wheel"/>
     <axis xyz="0 1 0"/>
+    <limit effort="10000" velocity="1000"/>
+    <dynamics damping="1.0" friction="1.0"/>
   </joint>
   <joint name="joint_2" type="revolute">
     <origin xyz="-0.15 0.2 0" rpy="0 0 0"/>
     <parent link="chassis"/>
-    <child link="back_right_wheel"/>
+    <child link="back_left_wheel"/>
     <axis xyz="0 1 0"/>
+    <limit effort="10000" velocity="1000"/>
+    <dynamics damping="1.0" friction="1.0"/>
   </joint>
   <joint name="joint_3" type="revolute">
     <origin xyz="-0.15 -0.2 0" rpy="0 0 0"/>
     <parent link="chassis"/>
-    <child link="front_left_wheel"/>
+    <child link="back_right_wheel"/>
     <axis xyz="0 1 0"/>
+    <limit effort="10000" velocity="1000"/>
+    <dynamics damping="1.0" friction="1.0"/>
+  </joint>
+  <joint name="joint_4" type="fixed">
+    <origin xyz="0 0 0.075" rpy="0 0 0"/>
+    <parent link="chassis"/>
+    <child link="lidar_base"/>
+    <axis xyz="0 0 1"/>
   </joint>
 </robot>

Commit message: Urdf correctionsand optimization / world.launch optimization

File: catkin_ws/src/my_robot/urdf/my_robot.xacro (robot description, xacro)
@@ -1,25 +1,29 @@
-<?xml version="1.0"?>
-<robot xmlns:xacro="http://www.ros.org/wiki/xacro" name="my_robot">
-    <link name='robot_footprint'></link>
-    <joint name="robot_footprint_joint" type="fixed">
-      <origin xyz="0 0 0" rpy="0 0 0" />
-      <parent link="robot_footprint"/>
-      <child link="chassis" />
-    </joint>
-   <link name='chassis'>
+<?xml version='1.0'?>
+ <robot name="my_robot" xmlns:xacro="http://www.ros.org/wiki/xacro">
+  <link name="robot_footprint"></link>
+  <joint name="robot_footprint_joint" type="fixed">
+    <origin xyz="0 0 0" rpy="0 0 0" />
+    <parent link="robot_footprint"/>
+    <child link="chassis" />
+  </joint>
+  <link name='chassis'>
     <pose>0 0 0.1 0 0 0</pose>
     <inertial>
       <mass value="15.0"/>
-      <origin xyz="0.0 0 0" rpy=" 0 0 0"/>
-      <inertia ixx="0.1" ixy="0" ixz="0" iyy="0.1" iyz="0" izz="0.1"/>
+      <origin xyz="0 0 0.1" rpy=" 0 0 0"/>
+      <inertia
+          ixx="0.1" ixy="0" ixz="0"
+          iyy="0.1" iyz="0"
+          izz="0.1"
+      />
     </inertial>
     <visual name='chassis_visual'>
-      <origin xyz="0 0 0" rpy=" 0 0 0"/>
+      <origin xyz="0 0 0.1" rpy=" 0 0 0"/>
       <geometry>
         <box size=".5 .3 .05"/>
       </geometry>
     </visual>
-    <collision name='chassis_collision'>
-      <origin xyz="0 0 0" rpy=" 0 0 0"/>
+    <collision name='collision'>
+      <origin xyz="0 0 0.1" rpy=" 0 0 0"/>
       <geometry>
         <box size=".5 .3 .05"/>
@@ -28,5 +32,4 @@
    </link>
    <link name='front_left_wheel'>
-    <pose>0 0 0.1 0 0 0</pose>
     <inertial>
       <mass value="1.0"/>
@@ -41,5 +44,5 @@
     </visual>
     <collision name='front_left_collision'>
-      <origin xyz="0 0 0" rpy=" 0 1.57050 1.5705"/>
+      <origin xyz="0 0 0" rpy=" 0 1.5705 1.5705"/>
       <geometry>
         <cylinder radius="0.1" length="0.1"/>
@@ -47,14 +50,17 @@
     </collision>
    </link>
+   <joint name="front_left_hinge" type="revolute">
+     <origin xyz="0.15 0.2 0.1" rpy="0 0 0"/>
+     <parent link="chassis"/>
+     <child link="front_left_wheel"/>
+     <axis xyz="0 1 0"/>
+     <limit effort="10000" velocity="1000"/>
+     <dynamics damping="1.0" friction="1.0"/>
+   </joint>
    <link name='front_right_wheel'>
-    <pose>0 0 0.1 0 0 0</pose>
     <inertial>
       <mass value="1.0"/>
       <origin xyz="0 0 0" rpy=" 0 1.5705 1.5705"/>
-      <inertia
-          ixx="0.1" ixy="0" ixz="0"
-          iyy="0.1" iyz="0"
-          izz="0.1"
-      />
+      <inertia ixx="0.1" ixy="0" ixz="0" iyy="0.1" iyz="0" izz="0.1"/>
     </inertial>
     <visual name='front_right_visual'>
@@ -71,6 +77,13 @@
     </collision>
    </link>
+   <joint name="front_right_hinge" type="revolute">
+     <origin xyz="0.15 -0.2 0.1" rpy="0 0 0"/>
+     <parent link="chassis"/>
+     <child link="front_right_wheel"/>
+     <axis xyz="0 1 0"/>
+     <limit effort="10000" velocity="1000"/>
+     <dynamics damping="1.0" friction="1.0"/>
+   </joint>
    <link name='back_left_wheel'>
-    <pose>0 0 0.1 0 0 0</pose>
     <inertial>
       <mass value="1.0"/>
@@ -91,14 +104,17 @@
     </collision>
    </link>
+   <joint name="back_left_hinge" type="revolute">
+     <origin xyz="-0.15 0.2 0.1" rpy="0 0 0"/>
+     <parent link="chassis"/>
+     <child link="back_left_wheel"/>
+     <axis xyz="0 1 0"/>
+     <limit effort="10000" velocity="1000"/>
+     <dynamics damping="1.0" friction="1.0"/>
+   </joint>
    <link name='back_right_wheel'>
-    <pose>0 0 0.1 0 0 0</pose>
     <inertial>
       <mass value="1.0"/>
       <origin xyz="0 0 0" rpy=" 1.5705 0 0"/>
-      <inertia
-          ixx="0.1" ixy="0" ixz="0"
-          iyy="0.1" iyz="0"
-          izz="0.1"
-      />
+      <inertia ixx="0.1" ixy="0" ixz="0" iyy="0.1" iyz="0" izz="0.1"/>
     </inertial>
     <visual name='back_right_visual'>
@@ -115,6 +131,13 @@
     </collision>
    </link>
+   <joint name="back_right_hinge" type="revolute">
+     <origin xyz="-0.15 -0.2 0.1" rpy="0 0 0"/>
+     <parent link="chassis"/>
+     <child link="back_right_wheel"/>
+     <axis xyz="0 1 0"/>
+     <limit effort="10000" velocity="1000"/>
+     <dynamics damping="1.0" friction="1.0"/>
+   </joint>
    <link name='lidar_base'>
-    <pose>0 0 0.1 0 0 0</pose>
     <inertial>
       <mass value="1.0"/>
@@ -128,5 +151,5 @@
       </geometry>
     </visual>
-    <collision name='lidar_base_collision'>
+   <collision name='lidar_base_collision'>
       <origin xyz="0 0 0" rpy=" 0 0 0"/>
       <geometry>
@@ -135,41 +158,9 @@
     </collision>
    </link>
-  <joint name="joint_0" type="revolute">
-    <origin xyz="0.15 0.2 0" rpy="0 0 0"/>
-    <parent link="chassis"/>
-    <child link="front_left_wheel"/>
-    <axis xyz="0 1 0"/>
-    <limit effort="10000" velocity="1000"/>
-    <dynamics damping="1.0" friction="1.0"/>
-  </joint>
-  <joint name="joint_1" type="revolute">
-    <origin xyz="0.15 -0.2 0" rpy="0 0 0"/>
-    <parent link="chassis"/>
-    <child link="front_right_wheel"/>
-    <axis xyz="0 1 0"/>
-    <limit effort="10000" velocity="1000"/>
-    <dynamics damping="1.0" friction="1.0"/>
-  </joint>
-  <joint name="joint_2" type="revolute">
-    <origin xyz="-0.15 0.2 0" rpy="0 0 0"/>
-    <parent link="chassis"/>
-    <child link="back_left_wheel"/>
-    <axis xyz="0 1 0"/>
-    <limit effort="10000" velocity="1000"/>
-    <dynamics damping="1.0" friction="1.0"/>
-  </joint>
-  <joint name="joint_3" type="revolute">
-    <origin xyz="-0.15 -0.2 0" rpy="0 0 0"/>
-    <parent link="chassis"/>
-    <child link="back_right_wheel"/>
-    <axis xyz="0 1 0"/>
-    <limit effort="10000" velocity="1000"/>
-    <dynamics damping="1.0" friction="1.0"/>
-  </joint>
-  <joint name="joint_4" type="fixed">
-    <origin xyz="0 0 0.075" rpy="0 0 0"/>
-    <parent link="chassis"/>
-    <child link="lidar_base"/>
-    <axis xyz="0 0 1"/>
-  </joint>
-</robot>
+   <joint name="lidar_link" type="fixed">
+     <origin xyz="0 0 0.175" rpy="0 0 0"/>
+     <parent link="chassis"/>
+     <child link="lidar_base"/>
+     <axis xyz="0 0 1"/>
+   </joint>
+ </robot>

Commit message: Robot colors and camera structure addition

File: catkin_ws/src/my_robot/urdf/my_robot.xacro (robot description, xacro)
@@ -1,4 +1,27 @@
 <?xml version='1.0'?>
  <robot name="my_robot" xmlns:xacro="http://www.ros.org/wiki/xacro">
+<!-- Color Definition -->
+  <gazebo reference="chassis">
+    <material>Gazebo/Orange</material>
+  </gazebo>
+  <gazebo reference="front_left_wheel">
+    <material>Gazebo/Black</material>
+  </gazebo>
+  <gazebo reference="front_right_wheel">
+    <material>Gazebo/Orange</material>
+  </gazebo>
+  <gazebo reference="back_left_wheel">
+    <material>Gazebo/Black</material>
+  </gazebo>
+  <gazebo reference="back_right_wheel">
+    <material>Gazebo/Black</material>
+  </gazebo>
+  <gazebo reference="lidar_base">
+    <material>Gazebo/White</material>
+  </gazebo>
+  <gazebo reference="camera">
+    <material>Gazebo/Black</material>
+  </gazebo>
+<!-- Robot Footprint -->
   <link name="robot_footprint"></link>
   <joint name="robot_footprint_joint" type="fixed">
@@ -7,4 +30,5 @@
     <child link="chassis" />
   </joint>
+<!-- Robot Chassis -->
   <link name='chassis'>
     <pose>0 0 0.1 0 0 0</pose>
@@ -12,9 +36,5 @@
       <mass value="15.0"/>
       <origin xyz="0 0 0.1" rpy=" 0 0 0"/>
-      <inertia
-          ixx="0.1" ixy="0" ixz="0"
-          iyy="0.1" iyz="0"
-          izz="0.1"
-      />
+      <inertia ixx="0.1" ixy="0" ixz="0" iyy="0.1" iyz="0" izz="0.1"/>
     </inertial>
     <visual name='chassis_visual'>
@@ -31,4 +51,5 @@
     </collision>
    </link>
+<!-- Robot Front Left Wheel Link-->
    <link name='front_left_wheel'>
     <inertial>
@@ -50,4 +71,5 @@
     </collision>
    </link>
+<!-- Robot Front Left Wheel Joint-->
    <joint name="front_left_hinge" type="revolute">
      <origin xyz="0.15 0.2 0.1" rpy="0 0 0"/>
@@ -58,4 +80,5 @@
      <dynamics damping="1.0" friction="1.0"/>
    </joint>
+<!-- Robot Front Right Wheel Link-->
    <link name='front_right_wheel'>
     <inertial>
@@ -77,4 +100,5 @@
     </collision>
    </link>
+<!-- Robot Front Right Wheel Joint-->
    <joint name="front_right_hinge" type="revolute">
      <origin xyz="0.15 -0.2 0.1" rpy="0 0 0"/>
@@ -85,4 +109,5 @@
      <dynamics damping="1.0" friction="1.0"/>
    </joint>
+<!-- Robot Back Left Wheel Link-->
    <link name='back_left_wheel'>
     <inertial>
@@ -104,4 +129,5 @@
     </collision>
    </link>
+<!-- Robot Back Left Wheel Joint-->
    <joint name="back_left_hinge" type="revolute">
      <origin xyz="-0.15 0.2 0.1" rpy="0 0 0"/>
@@ -112,4 +138,5 @@
      <dynamics damping="1.0" friction="1.0"/>
    </joint>
+<!-- Robot Back Right Wheel Link-->
    <link name='back_right_wheel'>
     <inertial>
@@ -131,4 +158,5 @@
     </collision>
    </link>
+<!-- Robot Back Right Wheel Joint-->
    <joint name="back_right_hinge" type="revolute">
      <origin xyz="-0.15 -0.2 0.1" rpy="0 0 0"/>
@@ -139,4 +167,5 @@
      <dynamics damping="1.0" friction="1.0"/>
    </joint>
+<!-- Lidar Base Link-->
    <link name='lidar_base'>
     <inertial>
@@ -158,4 +187,5 @@
     </collision>
    </link>
+<!-- Lidar Base Joint-->
    <joint name="lidar_link" type="fixed">
      <origin xyz="0 0 0.175" rpy="0 0 0"/>
@@ -164,3 +194,30 @@
      <axis xyz="0 0 1"/>
    </joint>
+<!-- Camera Link-->
+   <link name='camera'>
+    <inertial>
+      <mass value="0.1"/>
+      <origin xyz="0 0 0" rpy="0 0 0"/>
+      <inertia ixx="1e-6" ixy="0" ixz="0" iyy="1e-6" iyz="0" izz="1e-6"/>
+    </inertial>
+    <visual name='camera_visual'>
+      <origin xyz="0 0 0" rpy="0 0 0"/>
+      <geometry>
+        <box size=".025 .05 .05"/>
+      </geometry>
+    </visual>
+    <collision name='camera_collision'>
+      <origin xyz="0 0 0" rpy="0 0 0"/>
+      <geometry>
+        <box size=".025 .05 .05"/>
+      </geometry>
+    </collision>
+   </link>
+<!-- Camera Joint-->
+   <joint name="camera_link" type="fixed">
+     <origin xyz="0.25 0 0.1" rpy="0 0 0"/>
+     <parent link="chassis"/>
+     <child link="camera"/>
+     <axis xyz="0 1 0"/>
+   </joint>
  </robot>

Commit message: Lidar addition

File: catkin_ws/src/my_robot/urdf/my_robot.xacro (robot description, xacro)
@@ -6,5 +6,5 @@
   </gazebo>
   <gazebo reference="front_left_wheel">
-    <material>Gazebo/Black</material>
+    <material>Gazebo/Orange</material>
   </gazebo>
   <gazebo reference="front_right_wheel">
@@ -53,4 +53,5 @@
 <!-- Robot Front Left Wheel Link-->
    <link name='front_left_wheel'>
+    <pose>0 0 0.1 0 0 0</pose>
     <inertial>
       <mass value="1.0"/>
@@ -61,8 +62,8 @@
       <origin xyz="0 0 0" rpy=" 0 1.5705 1.5705"/>
       <geometry>
-        <cylinder radius="0.1" length="0.1"/>
-      </geometry>
-    </visual>
-    <collision name='front_left_collision'>
+         <cylinder radius="0.1" length="0.1"/>
+      </geometry>
+    </visual>
+    <collision name='collision'>
       <origin xyz="0 0 0" rpy=" 0 1.5705 1.5705"/>
       <geometry>
@@ -216,8 +217,35 @@
 <!-- Camera Joint-->
    <joint name="camera_link" type="fixed">
-     <origin xyz="0.25 0 0.1" rpy="0 0 0"/>
+     <origin xyz="0.26 0 0.1" rpy="0 0 0"/>
      <parent link="chassis"/>
      <child link="camera"/>
      <axis xyz="0 1 0"/>
    </joint>
+<!-- Lidar Link-->
+   <link name='hokuyo'>
+    <inertial>
+      <mass value="1e-5"/>
+      <origin xyz="0 0 0" rpy="0 0 0"/>
+      <inertia ixx="1e-6" ixy="0" ixz="0" iyy="1e-6" iyz="0" izz="1e-6"/>
+    </inertial>
+    <visual name='hokuyo_visual'>
+      <origin xyz="0 0 0" rpy="0 0 0"/>
+      <geometry>
+        <mesh filename="package://my_robot/meshes/hokuyo.dae"/>
+      </geometry>
+    </visual>
+    <collision name='hokuyo_collision'>
+      <origin xyz="0 0 0" rpy="0 0 0"/>
+      <geometry>
+        <box size=".1 .1 .1"/>
+      </geometry>
+    </collision>
+   </link>
+<!-- Lidar Joint-->
+   <joint name="hokuyo_link" type="fixed">
+     <origin xyz="0 0 0.25" rpy="0 0 0"/>
+     <parent link="chassis"/>
+     <child link="hokuyo"/>
+     <axis xyz="0 0 1"/>
+   </joint>
  </robot>

Commit message: Geometry color mistake corrected

File: catkin_ws/src/my_robot/urdf/my_robot.xacro (robot description, xacro)
@@ -6,8 +6,8 @@
   </gazebo>
   <gazebo reference="front_left_wheel">
-    <material>Gazebo/Orange</material>
+    <material>Gazebo/Black</material>
   </gazebo>
   <gazebo reference="front_right_wheel">
-    <material>Gazebo/Orange</material>
+    <material>Gazebo/Black</material>
   </gazebo>
   <gazebo reference="back_left_wheel">
@@ -59,5 +59,5 @@
       <inertia ixx="0.1" ixy="0" ixz="0" iyy="0.1" iyz="0" izz="0.1"/>
     </inertial>
-    <visual name='front_left_visual'>
+    <visual name='front_left_wheel_visual'>
       <origin xyz="0 0 0" rpy=" 0 1.5705 1.5705"/>
       <geometry>
@@ -88,5 +88,5 @@
       <inertia ixx="0.1" ixy="0" ixz="0" iyy="0.1" iyz="0" izz="0.1"/>
     </inertial>
-    <visual name='front_right_visual'>
+    <visual name='front_right_wheel_visual'>
       <origin xyz="0 0 0" rpy=" 0 1.5705 1.5705 "/>
       <geometry>
@@ -117,5 +117,5 @@
       <inertia ixx="0.1" ixy="0" ixz="0" iyy="0.1" iyz="0" izz="0.1"/>
     </inertial>
-    <visual name='back_left_visual'>
+    <visual name='back_left_wheel_visual'>
       <origin xyz="0 0 0" rpy=" 0 1.5705 1.5705"/>
       <geometry>
@@ -146,5 +146,5 @@
       <inertia ixx="0.1" ixy="0" ixz="0" iyy="0.1" iyz="0" izz="0.1"/>
     </inertial>
-    <visual name='back_right_visual'>
+    <visual name='back_right_wheel_visual'>
       <origin xyz="0 0 0" rpy=" 0 1.5705 1.5705"/>
       <geometry>

Commit message: Addition of Camera, Wheels and Lidar Plug-in

File: catkin_ws/src/my_robot/urdf/my_robot.xacro (robot description, xacro)
@@ -23,4 +23,5 @@
     <material>Gazebo/Black</material>
   </gazebo>
+  <xacro:include filename="$(find my_robot)/urdf/my_robot.gazebo" />
 <!-- Robot Footprint -->
   <link name="robot_footprint"></link>
@@ -73,5 +74,5 @@
    </link>
 <!-- Robot Front Left Wheel Joint-->
-   <joint name="front_left_hinge" type="revolute">
+   <joint name="front_left_hinge" type="continuous">
      <origin xyz="0.15 0.2 0.1" rpy="0 0 0"/>
      <parent link="chassis"/>
@@ -102,5 +103,5 @@
    </link>
 <!-- Robot Front Right Wheel Joint-->
-   <joint name="front_right_hinge" type="revolute">
+   <joint name="front_right_hinge" type="continuous">
      <origin xyz="0.15 -0.2 0.1" rpy="0 0 0"/>
      <parent link="chassis"/>
@@ -131,5 +132,5 @@
    </link>
 <!-- Robot Back Left Wheel Joint-->
-   <joint name="back_left_hinge" type="revolute">
+   <joint name="back_left_hinge" type="continuous">
      <origin xyz="-0.15 0.2 0.1" rpy="0 0 0"/>
      <parent link="chassis"/>
@@ -160,5 +161,5 @@
    </link>
 <!-- Robot Back Right Wheel Joint-->
-   <joint name="back_right_hinge" type="revolute">
+   <joint name="back_right_hinge" type="continuous">
      <origin xyz="-0.15 -0.2 0.1" rpy="0 0 0"/>
      <parent link="chassis"/>
